File: Aether/Aether.kicad_pcb (KiCad board)
At the start: 4 copper layers, 57.8 x 39.8 mm, 77 parts, among them IC1 DW3220TR13, IC2 nRF52833-QDAA-R, IC3 XC9290B16E0R-G, J1 USB_C_Receptacle_USB2.0, J2 NFC2, J3 NFC1, J4 Conn_ARM_JTAG_SWD_10, J5 Conn_01x02, J6 Conn_01x06, J7 Conn_01x02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

Commit message: Nuevo Aether
Parts:
- added Ctune3: 100pF, Capacitor_SMD:C_0805_2012Metric, F.Cu at (138.2, 83.4)
- added Ctune4: 100pF, Capacitor_SMD:C_0805_2012Metric, F.Cu at (138.2, 85.6)
- added Ctune5: 100pF, Capacitor_SMD:C_0805_2012Metric, F.Cu at (134.7, 83.5)
- added Ctune6: 100pF, Capacitor_SMD:C_0805_2012Metric, F.Cu at (134.7, 85.6)
- added RCC3: 1k, Resistor_SMD:R_0603_1608Metric, F.Cu at (140.9, 86.5)
- added RCCe1: 1k, Resistor_SMD:R_0603_1608Metric, F.Cu at (140.9, 82.6)
- AE1: value 2400-2500 MHz -> WE-MCA_7488910245
- RCC1, RCC2: footprint Resistor_SMD:R_0201_0603Metric -> Resistor_SMD:R_0603_1608Metric
- moved Ctune1 9.86 mm to (131.2, 83.2)
- moved Ctune2 9.63 mm to (131.2, 86.3), turned to -90 degrees
- moved R5 3.45 mm to (127.9, 91.0), turned to 0 degrees
- moved R7 3.04 mm to (128.8, 93.8), turned to 0 degrees
- moved R6 2.68 mm to (130.4, 90.0)
- moved S2 2.38 mm to (133.7, 90.6)
- moved S1 2.37 mm to (133.6, 93.8)
- moved C19 1.20 mm to (124.9, 83.9)
- moved E2 1.17 mm to (100.4, 95.5)
- moved E1 1.14 mm to (100.4, 74.7)
- moved RCC2 1.10 mm to (116.2, 95.4)
- moved RCC1 0.87 mm to (120.1, 95.3)
- moved C9 0.86 mm to (109.4, 93.6)
- moved C59 0.86 mm to (109.3, 90.5)
- moved C8 0.86 mm to (109.4, 92.1)
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Connections:
- IC2 pad 16: Net-(IC2-P0.18/NRESET) -> RESET
- IC2 pad 18: RESET -> VDD
- J2 pad 1: Net-(IC2-P0.10/NFC2) -> Net-(J2-Pin_1)
- J3 pad 1: Net-(IC2-P0.09/NFC1) -> Net-(J3-Pin_1)
- J4 pad 1: RESET -> VDD
- J4 pad 10: Net-(IC2-P0.18/NRESET) -> RESET
Routing:
- net Net-(IC2-P0.18/NRESET): track 30.6 -> 0.00 mm, vias 2 -> 0
- net RESET: track 65.0 -> 83.9 mm, vias 3 -> 5
- net Net-(IC2-P0.09/NFC1): track 23.3 -> 11.9 mm
- net Net-(IC2-P0.10/NFC2): track 22.5 -> 11.5 mm
- net WAKEUP: track 32.9 -> 39.2 mm
- net Net-(J3-Pin_1): track 0.00 -> 5.55 mm
- net Net-(J2-Pin_1): track 0.00 -> 5.25 mm
- net VDD: track 44.9 -> 48.7 mm
- net Net-(R5-Pad2): track 5.69 -> 3.31 mm
- net SPICLK: track 13.8 -> 15.9 mm
- net GND: track 40.8 -> 42.8 mm, vias 51 -> 125
- net Net-(Ctune3-Pad2): track 0.00 -> 1.64 mm
- net Net-(Ctune4-Pad2): track 0.00 -> 1.59 mm
- net SDA: track 31.8 -> 30.5 mm
- net Net-(J1-CC1): track 1.75 -> 2.82 mm
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Other:
- board text added: "λ"
