File: Aether/Aether.kicad_sch (KiCad schematic)
At the start: 77 parts, among them IC1 DW3220TR13, IC1 nRF52833-QDAA-R, IC3 XC9290B16E0R-G, J2 NFC2, J2 USB_C_Receptacle_USB2.0, J3 NFC1, J4 Conn_ARM_JTAG_SWD_10, J5 Conn_01x02, J6 Conn_01x06, J7 Conn_01x02, J8 Conn_01x03, Y1 ECS-320-8-47-CKM-TR3, Y1 ECS-384-10-33B-CKY-TR3, Y2 ECS-.327-9-12R-C-TR

Commit message: Nuevo Aether
Parts:
- added Ctune3, Ctune4, Ctune5, Ctune6: 100pF, Capacitor_SMD:C_0805_2012Metric, symbol Device:C
- added RCC3, RCCe1: 1k, Resistor_SMD:R_0603_1608Metric, symbol Device:R
- RCC1: renamed from RCC2; footprint Resistor_SMD:R_0201_0603Metric -> Resistor_SMD:R_0603_1608Metric
- RCC2: renamed from RCC1; footprint Resistor_SMD:R_0201_0603Metric -> Resistor_SMD:R_0603_1608Metric
- renumbered C18 to C10, C5 to C11, C12 to C14, C19 to C15, C13 to C16, C14 to C18, C9 to C19, C11 to C20, C2 to C21, C1 to C22, C3 to C23, C10 to C24, C4 to C25, C15 to C3, C16 to C4, C6 to C5, Ctune2 to Ctune1, Ctune1 to Ctune2, IC1 to IC2, J2 to J1, L4 to L1, L3 to L2, L1 to L3, L2 to L4, L2 to L5, Y1 to Y3
Connections:
- net GND: now also RCC3.1, RCCe1.2
- net RESET: now also IC2.16 (P0.18/NRESET), J4.10 (~{RESET}); no longer IC2.18 (VDD_2), J4.1 (VTref)
- net VDD: now also IC2.18 (VDD_2), J4.1 (VTref)
- net at Ctune2.1, IC2.22 (P0.09/NFC1): now also Ctune6.2; no longer J3.1 (Pin_1)
- net at Ctune1.1, IC2.23 (P0.10/NFC2): now also Ctune5.2; no longer J2.1 (Pin_1)
- new net: Ctune3.1, J2.1 (Pin_1), RCCe1.1
- new net: Ctune4.2, Ctune6.1
- new net: Ctune3.2, Ctune5.1
- new net: Ctune4.1, J3.1 (Pin_1), RCC3.2
Other:
- moved on the sheet: Ctune1, Ctune2, J2, J3
